Commit message: Python launch file, camera working. TODO: load plugins without env variables

File: src/models_pkg/rcCar_assembly/model.urdf.xacro (robot description, xacro)
@@ -4,14 +4,21 @@
   <xacro:include filename="$(find models_pkg)/wheel_right/model.urdf.xacro"/>
   <xacro:include filename="$(find models_pkg)/steering_column/model.urdf.xacro"/>
-  <link name="base_footprint" />
+  <!-- Default link -->
+  <link name="base_footprint">
+  </link>
   <joint
     name="base_footprint_joint" type="fixed">
-    <parent link="base_footprint" />
-    <child link="base_link" />
+    <parent link="base_link" />
+    <child link="base_footprint" />
     <origin xyz="0.0 0.0 0.0" rpy="0 0 1.5708" />
   </joint>
+  <gazebo reference="base_footprint_joint">
+    <disableFixedJointLumping>true</disableFixedJointLumping>
+    <preserveFixedJoint>true</preserveFixedJoint>
+  </gazebo>
   <!-- Chassis link -->
   <link name='base_link'>
       <inertial>
+        <origin rpy="0 0 -1.57079" xyz="0 0 -0.0065"/>
         <mass value="0.26244"/>
         <inertia ixx="0.00283444" ixy="0.0" ixz="0.0" iyy="0.00039867" iyz="0.0" izz="0.00323293"/>
@@ -31,41 +38,18 @@
           <box size="0.135 0.36 0.002"/>
         </geometry>
-        <surface>
-          <friction>
-            <ode>
-              <mu>1</mu>
-              <mu2>1</mu2>
-              <fdir1>0 0 0</fdir1>
-              <slip1>0</slip1>
-              <slip2>0</slip2>
-            </ode>
-            <torsional>
-              <coefficient>1</coefficient>
-              <patch_radius>0</patch_radius>
-              <surface_radius>0</surface_radius>
-              <use_patch_radius>1</use_patch_radius>
-              <ode>
-                <slip>0</slip>
-              </ode>
-            </torsional>
-          </friction>
-          <bounce>
-            <restitution_coefficient>0</restitution_coefficient>
-            <threshold>1e+06</threshold>
-          </bounce>
-        </surface>
       </collision>
     </link>
-  <!-- Left Wheel links -->
+  <!-- Left Wheel links and joints -->
   <xacro:wheel_left prefix="wheel_rear_left" x="-0.152" y="0.081" z="0" />
   <xacro:wheel_left prefix="wheel_front_left" x="0.118" y="0.081" z="0" />
   <xacro:steering_column prefix="steer_left" x="0.112" y="0.0725" z="0" z_joint="0.005" />
-  <!-- Right Wheel links -->
+  <!-- Right Wheel links and joints-->
   <xacro:wheel_right prefix="wheel_rear_right" x="-0.152" y="-0.081" z="0" />
   <xacro:wheel_right prefix="wheel_front_right" x="0.118" y="-0.081" z="0" />
   <xacro:steering_column prefix="steer_right" x="0.112" y="-0.0725" z="0" z_joint="-0.005" />
-  <!-- Car body link -->
+  <!-- Car body link and joint -->
   <link name='car_body_link'>
     <inertial>
+        <origin rpy="0 0 -1.57079" xyz="0 0.024 -0.028"/>
         <mass value="1"/>
         <inertia ixx="0.166667" ixy="0.0" ixz="0.0" iyy="0.166667" iyz="0.0" izz="0.166667"/>
@@ -77,4 +61,10 @@
       </geometry>
     </visual>
+    <collision>
+      <origin xyz="0 0 0" rpy="0 0 0"/>
+      <geometry>
+        <box size="0.2 0.4 0.1"/> <!-- approximate bounding box -->
+      </geometry>
+    </collision>
   </link>
   <joint name='car_body_joint' type='fixed'>
@@ -82,15 +72,123 @@
     <child link="car_body_link" />
     <origin xyz="0.0 0.0 0.0" rpy="0 0 0" />
+    <dynamics damping="0" friction="0" />
   </joint>
-<!--
-  <include>
-    <uri>model://camera</uri>
-    <origin rpy="0 0.2617 0" xyz="0 0 0.2"/>
-    <name>camera</name>
-  </include>
-  <joint name="joint_camera" type="fixed">
-    <parent link="chassis::link"/>
-    <child link="camera::link_camera"/>
-    <origin rpy="0 -0 0" xyz="0 0 0"/>
-  </joint> -->
+  <gazebo reference="car_body_joint">
+    <disableFixedJointLumping>true</disableFixedJointLumping>
+    <preserveFixedJoint>true</preserveFixedJoint>
+  </gazebo>
+  <!-- Camera link and joint -->
+  <link name="camera_link">
+    <inertial>
+        <origin xyz="0 0 0.2" rpy="0 0.2617 0" />
+        <mass value="0.0052875"/>
+        <inertia ixx="4.1e-07" ixy="0.0" ixz="0.0" iyy="7.9e-07" iyz="0.0" izz="4.1e-07"/>
+    </inertial>
+    <visual>
+      <origin xyz="0 0 0.2" rpy="0 0.2617 0" />
+      <geometry>
+        <box size="0.005 0.03 0.03" />
+      </geometry>
+      <material name="Grey">
+        <color rgba="0.7 0.7 0.7 1.0"/>
+      </material>
+    </visual>
+    <collision>
+        <origin xyz="0 0 0.2" rpy="0 0.2617 0" />
+        <geometry>
+          <box size="0.005 0.03 0.03"/>
+        </geometry>
+    </collision>
+  </link>
+  <joint name="camera_joint" type="fixed">
+    <parent link="base_link" />
+    <child link="camera_link" />
+    <origin xyz="0 0 0" rpy="0 0 -1.5708" />
+    <dynamics damping="0" friction="0" />
+  </joint>
+  <gazebo reference="camera_joint">
+    <disableFixedJointLumping>true</disableFixedJointLumping>
+    <preserveFixedJoint>true</preserveFixedJoint>
+  </gazebo>
+  <!-- Gazebo plugins -->
+  <!-- Camera Plugin -->
+  <gazebo reference="camera_link">
+    <sensor type="camera" name="camera1">
+      <pose>0 0 0.2 0 0.2617 0</pose>
+      <always_on>true</always_on>
+      <update_rate>30.0</update_rate>
+      <visualize>true</visualize>
+      <camera>
+        <horizontal_fov>1.085594795</horizontal_fov>
+        <image>
+          <width>640</width>
+          <height>480</height>
+          <format>R8G8B8</format>
+        </image>
+        <clip>
+          <near>0.02</near>
+          <far>100</far>
+        </clip>
+        <noise>
+          <type>gaussian</type>
+          <mean>0.0</mean>
+          <stddev>0.0</stddev>
+        </noise>
+      </camera>
+      <plugin name="camera_controller" filename="libgazebo_ros_camera.so">
+        <baseline>0.2</baseline>
+        <alwaysOn>true</alwaysOn>
+        <updateRate>30.0</updateRate>
+        <imageTopicName>image_raw</imageTopicName>
+        <cameraInfoTopicName>camera_info</cameraInfoTopicName>
+        <frameName>camera_link</frameName>
+        <hackBaseline>0.0</hackBaseline>
+        <distortionK1>0.0</distortionK1>
+        <distortionK2>0.0</distortionK2>
+        <distortionK3>0.0</distortionK3>
+        <distortionT1>0.0</distortionT1>
+        <distortionT2>0.0</distortionT2>
+        <robotNamespace>/</robotNamespace>
+      </plugin>
+    </sensor>
+  </gazebo>
+  <!-- Car-like robot Plugin -->
+  <gazebo>
+    <plugin name="CarLikeRobotPlugin" filename="libcar_plugin.so">
+      <wheelbase>0.26</wheelbase>
+      <axletrack>0.162</axletrack>
+      <wheelradius>0.0325</wheelradius>
+      <speed_wheel_joints>
+        <front_wheel_joints>
+          <leftjoint>wheel_front_left_joint</leftjoint>
+          <rightjoint>wheel_front_right_joint</rightjoint>
+        </front_wheel_joints>
+        <rear_wheel_joints>
+          <leftjoint>wheel_rear_left_joint</leftjoint>
+          <rightjoint>wheel_rear_right_joint</rightjoint>
+        </rear_wheel_joints>
+        <kp>0.01</kp>
+        <ki>0.0</ki>
+        <kd>0.0</kd>
+      </speed_wheel_joints>
+      <steer_wheel_joints>
+        <leftjoint>steer_left_joint</leftjoint>
+        <rightjoint>steer_right_joint</rightjoint>
+        <kp>10</kp>
+        <ki>0.0</ki>
+        <kd>0.1</kd>
+      </steer_wheel_joints>
+      <initial_steer>0.0</initial_steer>
+      <initial_speed>0.0</initial_speed>
+      <robotNamespace>/</robotNamespace>
+    </plugin>
+  </gazebo>
+  <!-- BNO055 IMU Plugin  -->
+  <gazebo>
+    <plugin name="bno055" filename="libbno055_plugin.so"/>
+  </gazebo>
+  <!-- GPS Plugin -->
+  <gazebo>
+    <plugin name="gps" filename="libgps_plugin.so"/>
+  </gazebo>
 </robot>

Commit message: Model editing, the car is stable in simulation.

File: src/models_pkg/rcCar_assembly/model.urdf.xacro (robot description, xacro)
@@ -11,5 +11,5 @@
     <parent link="base_link" />
     <child link="base_footprint" />
-    <origin xyz="0.0 0.0 0.0" rpy="0 0 1.5708" />
+    <origin xyz="0.0 0.0 0.0" rpy="0 0 0" />
   </joint>
   <gazebo reference="base_footprint_joint">
@@ -20,10 +20,9 @@
   <link name='base_link'>
       <inertial>
-        <origin rpy="0 0 -1.57079" xyz="0 0 -0.0065"/>
         <mass value="0.26244"/>
-        <inertia ixx="0.00283444" ixy="0.0" ixz="0.0" iyy="0.00039867" iyz="0.0" izz="0.00323293"/>
+        <inertia ixx="0.002" ixy="0.0" ixz="0.0" iyy="0.002" iyz="0.0" izz="0.002"/>
       </inertial>
       <visual>
-        <origin rpy="0 0 -1.57079" xyz="0 0 -0.0065"/>
+        <origin rpy="0 0 0" xyz="0 0 0"/>
         <geometry>
           <mesh filename="package://models_pkg/chassis/meshes/chassisV5.dae"/>
@@ -38,23 +37,67 @@
           <box size="0.135 0.36 0.002"/>
         </geometry>
+        <surface>
+          <friction>
+            <ode>
+              <mu>1</mu>
+              <mu2>1</mu2>
+              <fdir1>0 0 0</fdir1>
+              <slip1>0</slip1>
+              <slip2>0</slip2>
+            </ode>
+            <torsional>
+              <coefficient>1</coefficient>
+              <patch_radius>0</patch_radius>
+              <surface_radius>0</surface_radius>
+              <use_patch_radius>1</use_patch_radius>
+              <ode>
+                <slip>0</slip>
+              </ode>
+            </torsional>
+          </friction>
+          <bounce>
+            <restitution_coefficient>0</restitution_coefficient>
+            <threshold>1e+06</threshold>
+          </bounce>
+          <contact>
+            <collide_without_contact>0</collide_without_contact>
+            <collide_without_contact_bitmask>1</collide_without_contact_bitmask>
+            <collide_bitmask>1</collide_bitmask>
+            <ode>
+              <soft_cfm>0</soft_cfm>
+              <soft_erp>0.2</soft_erp>
+              <kp>1e+6</kp>
+              <kd>1</kd>
+              <max_vel>0.01</max_vel>
+              <min_depth>0</min_depth>
+            </ode>
+            <!-- <bullet>
+              <split_impulse>1</split_impulse>
+              <split_impulse_penetration_threshold>-0.01</split_impulse_penetration_threshold>
+              <soft_cfm>0</soft_cfm>
+              <soft_erp>0.2</soft_erp>
+              <kp>1e+13</kp>
+              <kd>1</kd>
+            </bullet> -->
+          </contact>
+        </surface>
       </collision>
     </link>
   <!-- Left Wheel links and joints -->
-  <xacro:wheel_left prefix="wheel_rear_left" x="-0.152" y="0.081" z="0" />
-  <xacro:wheel_left prefix="wheel_front_left" x="0.118" y="0.081" z="0" />
-  <xacro:steering_column prefix="steer_left" x="0.112" y="0.0725" z="0" z_joint="0.005" />
+  <xacro:wheel_left prefix="wheel_rear_left" x="-0.152" y="0.081" z="-0.033" />
+  <xacro:wheel_left prefix="wheel_front_left" x="0.118" y="0.081" z="-0.033" />
+  <!-- <xacro:steering_column prefix="steer_left" x="0.112" y="0.0725" z="0" z_joint="0.005" /> -->
   <!-- Right Wheel links and joints-->
-  <xacro:wheel_right prefix="wheel_rear_right" x="-0.152" y="-0.081" z="0" />
-  <xacro:wheel_right prefix="wheel_front_right" x="0.118" y="-0.081" z="0" />
-  <xacro:steering_column prefix="steer_right" x="0.112" y="-0.0725" z="0" z_joint="-0.005" />
+  <xacro:wheel_right prefix="wheel_rear_right" x="-0.152" y="-0.081" z="-0.033" />
+  <xacro:wheel_right prefix="wheel_front_right" x="0.118" y="-0.081" z="-0.033" />
+  <!-- <xacro:steering_column prefix="steer_right" x="0.112" y="-0.0725" z="0" z_joint="0.005" /> -->
   <!-- Car body link and joint -->
   <link name='car_body_link'>
     <inertial>
-        <origin rpy="0 0 -1.57079" xyz="0 0.024 -0.028"/>
         <mass value="1"/>
         <inertia ixx="0.166667" ixy="0.0" ixz="0.0" iyy="0.166667" iyz="0.0" izz="0.166667"/>
     </inertial>
     <visual name='visual'>
-      <origin rpy="0 0 -1.57079" xyz="0 0.024 -0.028"/>
+      <origin rpy="0 0 0" xyz="-0.024 0 -0.028"/>
       <geometry>
         <mesh filename="package://models_pkg/car_body/meshes/CarBody.dae"/>
@@ -81,5 +124,4 @@
   <link name="camera_link">
     <inertial>
-        <origin xyz="0 0 0.2" rpy="0 0.2617 0" />
         <mass value="0.0052875"/>
         <inertia ixx="4.1e-07" ixy="0.0" ixz="0.0" iyy="7.9e-07" iyz="0.0" izz="4.1e-07"/>
@@ -104,5 +146,5 @@
     <parent link="base_link" />
     <child link="camera_link" />
-    <origin xyz="0 0 0" rpy="0 0 -1.5708" />
+    <origin xyz="0 0 0" rpy="0 0 0" />
     <dynamics damping="0" friction="0" />
   </joint>
@@ -154,5 +196,5 @@
   </gazebo>
   <!-- Car-like robot Plugin -->
-  <gazebo>
+  <!-- <gazebo>
     <plugin name="CarLikeRobotPlugin" filename="libcar_plugin.so">
       <wheelbase>0.26</wheelbase>
@@ -183,12 +225,12 @@
       <robotNamespace>/</robotNamespace>
     </plugin>
-  </gazebo>
+  </gazebo> -->
   <!-- BNO055 IMU Plugin  -->
-  <gazebo>
+  <!-- <gazebo>
     <plugin name="bno055" filename="libbno055_plugin.so"/>
-  </gazebo>
+  </gazebo> -->
   <!-- GPS Plugin -->
-  <gazebo>
+  <!-- <gazebo>
     <plugin name="gps" filename="libgps_plugin.so"/>
-  </gazebo>
+  </gazebo> -->
 </robot>

File: src/models_pkg/steering_column/model.urdf.xacro (robot description, xacro)
@@ -7,5 +7,5 @@
             </inertial>
             <visual>
-                <origin rpy="0 0 0" xyz="${x} ${y} ${z}"/>
+                <origin rpy="0 0 1.5708" xyz="${x} ${y} ${z}"/>
                 <geometry>
                     <cylinder radius="0.001" length="0.01" />
@@ -13,5 +13,5 @@
             </visual>
             <collision>
-                <origin xyz="${x} ${y} ${z}" rpy="0 0 0" />
+                <origin xyz="0 0 0" rpy="0 0 0" />
                 <geometry>
                     <cylinder radius="0.001" length="0.01" />
@@ -40,5 +40,26 @@
                         <threshold>1e+06</threshold>
                     </bounce>
-                </surface>
+                    <contact>
+                        <collide_without_contact>0</collide_without_contact>
+                        <collide_without_contact_bitmask>1</collide_without_contact_bitmask>
+                        <collide_bitmask>1</collide_bitmask>
+                        <ode>
+                        <soft_cfm>0</soft_cfm>
+                        <soft_erp>0.2</soft_erp>
+                        <kp>1e+13</kp>
+                        <kd>1</kd>
+                        <max_vel>0.01</max_vel>
+                        <min_depth>0</min_depth>
+                        </ode>
+                        <bullet>
+                        <split_impulse>1</split_impulse>
+                        <split_impulse_penetration_threshold>-0.01</split_impulse_penetration_threshold>
+                        <soft_cfm>0</soft_cfm>
+                        <soft_erp>0.2</soft_erp>
+                        <kp>1e+13</kp>
+                        <kd>1</kd>
+                        </bullet>
+                    </contact>
+                    </surface>
             </collision>
         </link>
@@ -49,5 +70,5 @@
             <parent link="base_link" />
             <child link="${prefix}_link" />
-            <origin xyz="0 0 ${z_joint}" rpy="0 -0 -1.5708" />
+            <origin xyz="0 0 ${z_joint}" rpy="0 -0 0" />
             <axis xyz="0 1 0"/>
             <limit upper="1.79769e+308" lower="-1.79769e+308" effort="1" velocity="-1" />

File: src/models_pkg/wheel_left/model.urdf.xacro (robot description, xacro)
@@ -4,8 +4,8 @@
             <inertial>
                 <mass value="0.038"/>
-                <inertia ixx="0.00001283" ixy="0.0" ixz="0.0" iyy="0.00001283" iyz="0.0" izz="0.00002069"/>
+                <inertia ixx="0.00003" ixy="0.0" ixz="0.0" iyy="0.00003" iyz="0.0"  izz="0.00003"/>
             </inertial>
             <visual>
-                <origin rpy="0 0 0" xyz="${x} ${y} ${z}"/>
+                <origin rpy="0 0 0" xyz="0 0 0"/>
                 <geometry>
                     <mesh filename="package://models_pkg/wheel_left/meshes/rim.dae"/>
@@ -13,18 +13,18 @@
             </visual>
             <collision>
-                <origin xyz="${x} ${y} ${z}" rpy="0 0 0" />
+                <origin xyz="0 0 0" rpy="0 0 0" />
                 <geometry>
-                    <cylinder radius="0.33000" length="0.28000" />
+                    <cylinder radius="0.033" length="0.028" />
                 </geometry>
                 <surface>
                     <friction>
                         <ode>
-                        <mu>0.7</mu>
-                        <mu2>0.7</mu2>
-                        <fdir1>0 0 0</fdir1>
-                        <slip1>0</slip1>
-                        <slip2>0</slip2>
+                            <mu>0.7</mu>
+                            <mu2>0.7</mu2>
+                            <fdir1>0 0 0</fdir1>
+                            <slip1>0</slip1>
+                            <slip2>0</slip2>
                         </ode>
-                        <torsional>
+                        <!-- <torsional>
                         <coefficient>1</coefficient>
                         <patch_radius>0</patch_radius>
@@ -34,5 +34,5 @@
                             <slip>0</slip>
                         </ode>
-                        </torsional>
+                        </torsional> -->
                     </friction>
                     <bounce>
@@ -40,4 +40,25 @@
                         <threshold>1e+06</threshold>
                     </bounce>
+                    <contact>
+                        <collide_without_contact>0</collide_without_contact>
+                        <collide_without_contact_bitmask>1</collide_without_contact_bitmask>
+                        <collide_bitmask>1</collide_bitmask>
+                        <ode>
+                        <soft_cfm>0</soft_cfm>
+                        <soft_erp>0.2</soft_erp>
+                        <kp>1e+07</kp>
+                        <kd>1</kd>
+                        <max_vel>0.01</max_vel>
+                        <min_depth>0</min_depth>
+                        </ode>
+                        <!-- <bullet>
+                        <split_impulse>1</split_impulse>
+                        <split_impulse_penetration_threshold>-0.01</split_impulse_penetration_threshold>
+                        <soft_cfm>0</soft_cfm>
+                        <soft_erp>0.2</soft_erp>
+                        <kp>1e+07</kp>
+                        <kd>1</kd>
+                        </bullet> -->
+                    </contact>
                 </surface>
             </collision>
@@ -46,9 +67,9 @@
             define a continuous joint to allow the wheels to freely rotate about
             an axis -->
-        <joint name="${prefix}_joint" type="revolute">
+        <joint name="${prefix}_joint" type="continuous">
             <parent link="base_link" />
             <child link="${prefix}_link" />
-            <origin xyz="0 0 0" rpy="0 -0 -1.5708" />
-            <axis xyz="0 0 -1"/>
+            <origin xyz="${x} ${y} ${z}" rpy="0 0 0" />
+            <axis xyz="0 1 0"/>
             <limit upper="1.79769e+308" lower="-1.79769e+308" effort="1" velocity="-1" />
             <dynamics damping="0" friction="0" />

File: src/models_pkg/wheel_right/model.urdf.xacro (robot description, xacro)
@@ -4,26 +4,16 @@
             <inertial>
                 <mass value="0.038"/>
-                <inertia ixx="0.00001283" ixy="0.0" ixz="0.0" iyy="0.00001283" iyz="0.0" izz="0.00002069"/>
+                <inertia ixx="0.00003" ixy="0.0" ixz="0.0" iyy="0.00003" iyz="0.0"  izz="0.00003"/>
             </inertial>
             <visual>
-                <origin rpy="0 0 0" xyz="${x} ${y} ${z}"/>
+                <origin rpy="0 0 0" xyz="0 0 0"/>
                 <geometry>
                     <mesh filename="package://models_pkg/wheel_right/meshes/rim.dae"/>
                 </geometry>
-                <!-- <material name="wheel_right">
-                    <lighting>1</lighting>
-                    <shader type='vertex'>
-                        <normal_map>__default__</normal_map>
-                    </shader>
-                    <ambient>0.2 0.2 0.2 1</ambient>
-                    <diffuse>0.3 0.3 0.3 1</diffuse>
-                    <specular>0.5 0.5 0.5 1</specular>
-                    <emissive>0.0 0.0 0.0 0.0</emissive>
-                </material> -->
             </visual>
             <collision>
-                <origin xyz="${x} ${y} ${z}" rpy="0 0 0" />
+                <origin xyz="0 0 0" rpy="0 0 0" />
                 <geometry>
-                    <cylinder radius="0.33000" length="0.28000" />
+                    <cylinder radius="0.033" length="0.028" />
                 </geometry>
                 <surface>
@@ -36,5 +26,5 @@
                         <slip2>0</slip2>
                         </ode>
-                        <torsional>
+                        <!-- <torsional>
                         <coefficient>1</coefficient>
                         <patch_radius>0</patch_radius>
@@ -44,5 +34,5 @@
                             <slip>0</slip>
                         </ode>
-                        </torsional>
+                        </torsional> -->
                     </friction>
                     <bounce>
@@ -50,5 +40,26 @@
                         <threshold>1e+06</threshold>
                     </bounce>
-                </surface>
+                    <contact>
+                        <collide_without_contact>0</collide_without_contact>
+                        <collide_without_contact_bitmask>1</collide_without_contact_bitmask>
+                        <collide_bitmask>1</collide_bitmask>
+                        <ode>
+                        <soft_cfm>0</soft_cfm>
+                        <soft_erp>0.2</soft_erp>
+                        <kp>1e+07</kp>
+                        <kd>1</kd>
+                        <max_vel>0.01</max_vel>
+                        <min_depth>0</min_depth>
+                        </ode>
+                        <!-- <bullet>
+                        <split_impulse>1</split_impulse>
+                        <split_impulse_penetration_threshold>-0.01</split_impulse_penetration_threshold>
+                        <soft_cfm>0</soft_cfm>
+                        <soft_erp>0.2</soft_erp>
+                        <kp>1e+07</kp>
+                        <kd>1</kd>
+                        </bullet> -->
+                    </contact>
+                    </surface>
             </collision>
         </link>
@@ -56,10 +67,10 @@
             define a continuous joint to allow the wheels to freely rotate about
             an axis -->
-        <joint name="${prefix}_joint" type="revolute">
+        <joint name="${prefix}_joint" type="continuous">
             <parent link="base_link" />
             <child link="${prefix}_link" />
             <!-- change sign of yaw if fornt and rear are not right -->
-            <origin xyz="0 0 0" rpy="0 -0 -1.5708" />
-            <axis xyz="0 0 -1"/>
+            <origin xyz="${x} ${y} ${z}" rpy="0 -0 0" />
+            <axis xyz="0 1 0"/>
             <limit upper="1.79769e+308" lower="-1.79769e+308" effort="1" velocity="-1" />
             <dynamics damping="0" friction="0" />
