Commit message: Minor model changes for collision boxes

File: src/models_pkg/rcCar_assembly/model.urdf.xacro (robot description, xacro)
@@ -33,5 +33,5 @@
       </visual>
       <collision>
-        <origin rpy="0 0 0" xyz="0 0 0"/>
+        <origin rpy="0 0 0" xyz="0 0 1.5709"/>
         <geometry>
           <box size="0.135 0.36 0.002"/>
@@ -85,11 +85,11 @@
     </link>
   <!-- Left Wheel links and joints -->
-  <xacro:wheel_left prefix="wheel_rear_left" x="-0.152" y="0.081" z="-0.033" />
-  <xacro:wheel_left prefix="wheel_front_left" x="0.118" y="0.081" z="-0.033" />
-  <!-- <xacro:steering_column prefix="steer_left" x="0.112" y="0.0725" z="0" z_joint="0.005" /> -->
+  <xacro:steering_column prefix="steer_left" x="0.112" y="0.0725" z="-0.0165" z_joint="0.005" />
+  <xacro:wheel_left prefix="wheel_rear_left" x="-0.152" y="0.081" z="-0.0165" parent="base_link" />
+  <xacro:wheel_left prefix="wheel_front_left" x="0.118" y="0.081" z="-0.0165" parent="steer_left_link" />
   <!-- Right Wheel links and joints-->
-  <xacro:wheel_right prefix="wheel_rear_right" x="-0.152" y="-0.081" z="-0.033" />
-  <xacro:wheel_right prefix="wheel_front_right" x="0.118" y="-0.081" z="-0.033" />
-  <!-- <xacro:steering_column prefix="steer_right" x="0.112" y="-0.0725" z="0" z_joint="0.005" /> -->
+  <xacro:steering_column prefix="steer_right" x="0.112" y="-0.0725" z="-0.0165" z_joint="0.005" />
+  <xacro:wheel_right prefix="wheel_rear_right" x="-0.152" y="-0.081" z="-0.0165" parent="base_link" />
+  <xacro:wheel_right prefix="wheel_front_right" x="0.118" y="-0.081" z="-0.0165" parent="steer_right_link" />
   <!-- Car body link and joint -->
   <link name='car_body_link'>
@@ -104,8 +104,8 @@
       </geometry>
     </visual>
-    <collision>
-      <origin xyz="0 0 0" rpy="0 0 0"/>
+    <collision >
+      <origin xyz="-0.024 0 0.07" rpy="0 0 1.5709"/>
       <geometry>
-        <box size="0.2 0.4 0.1"/> <!-- approximate bounding box -->
+        <box size="0.2 0.5 0.1"/>
       </geometry>
     </collision>
@@ -196,5 +196,5 @@
   </gazebo>
   <!-- Car-like robot Plugin -->
-  <!-- <gazebo>
+  <gazebo>
     <plugin name="CarLikeRobotPlugin" filename="libcar_plugin.so">
       <wheelbase>0.26</wheelbase>
@@ -225,5 +225,5 @@
       <robotNamespace>/</robotNamespace>
     </plugin>
-  </gazebo> -->
+  </gazebo>
   <!-- BNO055 IMU Plugin  -->
   <!-- <gazebo>

File: src/models_pkg/steering_column/model.urdf.xacro (robot description, xacro)
@@ -3,9 +3,9 @@
         <link name="${prefix}_link">
             <inertial>
-                <mass value="0.001"/>
-                <inertia ixx="0.00014583" ixy="0.0" ixz="0.0" iyy="0.00014583" iyz="0.0" izz="0.000125"/>
+                <mass value="0.05"/>
+                <inertia ixx="1e-5" ixy="0.0" ixz="0.0"  iyy="1e-5" iyz="0.0" izz="1e-5"/>
             </inertial>
             <visual>
-                <origin rpy="0 0 1.5708" xyz="${x} ${y} ${z}"/>
+                <origin rpy="0 0 0" xyz="${x} ${y} ${z}"/>
                 <geometry>
                     <cylinder radius="0.001" length="0.01" />
@@ -47,5 +47,5 @@
                         <soft_cfm>0</soft_cfm>
                         <soft_erp>0.2</soft_erp>
-                        <kp>1e+13</kp>
+                        <kp>1e+6</kp>
                         <kd>1</kd>
                         <max_vel>0.01</max_vel>
@@ -57,5 +57,5 @@
                         <soft_cfm>0</soft_cfm>
                         <soft_erp>0.2</soft_erp>
-                        <kp>1e+13</kp>
+                        <kp>1e+6</kp>
                         <kd>1</kd>
                         </bullet>
@@ -71,7 +71,9 @@
             <child link="${prefix}_link" />
             <origin xyz="0 0 ${z_joint}" rpy="0 -0 0" />
-            <axis xyz="0 1 0"/>
-            <limit upper="1.79769e+308" lower="-1.79769e+308" effort="1" velocity="-1" />
-            <dynamics damping="0" friction="0" />
+            <axis xyz="0 0 1"/>
+             <!-- reasonable limits: ±30° -->
+            <limit lower="-0.6" upper="0.6" effort="10" velocity="5"/>
+            <!-- some damping -->
+            <dynamics damping="1.0" friction="0.1"/>
         </joint>
     </xacro:macro>

File: src/models_pkg/wheel_left/model.urdf.xacro (robot description, xacro)
@@ -1,4 +1,4 @@
-<robot xmlns:xacro="http://www.ros.org/wiki/xacro">
-    <xacro:macro name="wheel_left" params="prefix x y z">
+<robot xmlns:xacro="http://ros.org/wiki/xacro">
+    <xacro:macro name="wheel_left" params="prefix x y z parent">
         <link name="${prefix}_link">
             <inertial>
@@ -13,5 +13,5 @@
             </visual>
             <collision>
-                <origin xyz="0 0 0" rpy="0 0 0" />
+                <origin xyz="0 0 0" rpy="1.5709 0 0" />
                 <geometry>
                     <cylinder radius="0.033" length="0.028" />
@@ -68,5 +68,5 @@
             an axis -->
         <joint name="${prefix}_joint" type="continuous">
-            <parent link="base_link" />
+            <parent link="${parent}" />
             <child link="${prefix}_link" />
             <origin xyz="${x} ${y} ${z}" rpy="0 0 0" />

File: src/models_pkg/wheel_right/model.urdf.xacro (robot description, xacro)
@@ -1,4 +1,4 @@
-<robot xmlns:xacro="http://www.ros.org/wiki/xacro">
-    <xacro:macro name="wheel_right" params="prefix x y z">
+<robot xmlns:xacro="http://ros.org/wiki/xacro">
+    <xacro:macro name="wheel_right" params="prefix x y z parent">
         <link name="${prefix}_link">
             <inertial>
@@ -13,5 +13,5 @@
             </visual>
             <collision>
-                <origin xyz="0 0 0" rpy="0 0 0" />
+                <origin xyz="0 0 0" rpy="1.5709 0 0" />
                 <geometry>
                     <cylinder radius="0.033" length="0.028" />
@@ -68,5 +68,5 @@
             an axis -->
         <joint name="${prefix}_joint" type="continuous">
-            <parent link="base_link" />
+            <parent link="${parent}" />
             <child link="${prefix}_link" />
             <!-- change sign of yaw if fornt and rear are not right -->
