Commit message: Fixed car drift while stationary.

File: src/models_pkg/wheel_left/model.urdf.xacro (robot description, xacro)
@@ -15,5 +15,5 @@
                 <origin xyz="0 0 0" rpy="1.5709 0 0" />
                 <geometry>
-                    <cylinder radius="0.033" length="0.028" />
+                    <cylinder radius="0.0325" length="0.028" />
                 </geometry>
                 <surface>
@@ -47,6 +47,6 @@
                         <soft_cfm>0</soft_cfm>
                         <soft_erp>0.2</soft_erp>
-                        <kp>1e+07</kp>
-                        <kd>1</kd>
+                        <kp>1e+05</kp>
+                        <kd>10</kd>
                         <max_vel>0.01</max_vel>
                         <min_depth>0</min_depth>
@@ -72,6 +72,7 @@
             <origin xyz="${x} ${y} ${z}" rpy="0 0 0" />
             <axis xyz="0 1 0"/>
-            <limit upper="1.79769e+308" lower="-1.79769e+308" effort="1" velocity="-1" />
-            <dynamics damping="0" friction="0" />
+            <limit effort="10" velocity="100" />
+            <!-- <limit upper="1.79769e+308" lower="-1.79769e+308" effort="1" velocity="-1" /> -->
+            <dynamics damping="0.01" friction="0.01"/>
         </joint>
     </xacro:macro>

File: src/models_pkg/wheel_right/model.urdf.xacro (robot description, xacro)
@@ -15,5 +15,5 @@
                 <origin xyz="0 0 0" rpy="1.5709 0 0" />
                 <geometry>
-                    <cylinder radius="0.033" length="0.028" />
+                    <cylinder radius="0.0325" length="0.028" />
                 </geometry>
                 <surface>
@@ -47,6 +47,6 @@
                         <soft_cfm>0</soft_cfm>
                         <soft_erp>0.2</soft_erp>
-                        <kp>1e+07</kp>
-                        <kd>1</kd>
+                        <kp>1e+05</kp>
+                        <kd>10</kd>
                         <max_vel>0.01</max_vel>
                         <min_depth>0</min_depth>
@@ -73,6 +73,7 @@
             <origin xyz="${x} ${y} ${z}" rpy="0 -0 0" />
             <axis xyz="0 1 0"/>
-            <limit upper="1.79769e+308" lower="-1.79769e+308" effort="1" velocity="-1" />
-            <dynamics damping="0" friction="0" />
+            <limit effort="10" velocity="100" />
+            <!-- <limit upper="1.79769e+308" lower="-1.79769e+308" effort="1" velocity="-1" /> -->
+            <dynamics damping="0.01" friction="0.01"/>
         </joint>
     </xacro:macro>

Commit message: Fixed wheel drift, again.

File: src/models_pkg/wheel_left/model.urdf.xacro (robot description, xacro)
@@ -3,5 +3,5 @@
         <link name="${prefix}_link">
             <inertial>
-                <mass value="0.038"/>
+                <mass value="0.1"/>
                 <inertia ixx="0.00003" ixy="0.0" ixz="0.0" iyy="0.00003" iyz="0.0"  izz="0.00003"/>
             </inertial>
@@ -27,11 +27,11 @@
                         </ode>
                         <!-- <torsional>
-                        <coefficient>1</coefficient>
-                        <patch_radius>0</patch_radius>
-                        <surface_radius>0</surface_radius>
-                        <use_patch_radius>1</use_patch_radius>
-                        <ode>
-                            <slip>0</slip>
-                        </ode>
+                            <coefficient>1</coefficient>
+                            <patch_radius>0</patch_radius>
+                            <surface_radius>0</surface_radius>
+                            <use_patch_radius>1</use_patch_radius>
+                            <ode>
+                                <slip>0</slip>
+                            </ode>
                         </torsional> -->
                     </friction>

File: src/models_pkg/wheel_right/model.urdf.xacro (robot description, xacro)
@@ -3,5 +3,5 @@
         <link name="${prefix}_link">
             <inertial>
-                <mass value="0.038"/>
+                <mass value="0.1"/>
                 <inertia ixx="0.00003" ixy="0.0" ixz="0.0" iyy="0.00003" iyz="0.0"  izz="0.00003"/>
             </inertial>
@@ -23,15 +23,16 @@
                         <mu2>0.7</mu2>
                         <fdir1>0 0 0</fdir1>
+                        <!-- 0 0 0 -->
                         <slip1>0</slip1>
                         <slip2>0</slip2>
                         </ode>
                         <!-- <torsional>
-                        <coefficient>1</coefficient>
-                        <patch_radius>0</patch_radius>
-                        <surface_radius>0</surface_radius>
-                        <use_patch_radius>1</use_patch_radius>
-                        <ode>
-                            <slip>0</slip>
-                        </ode>
+                            <coefficient>1</coefficient>
+                            <patch_radius>0</patch_radius>
+                            <surface_radius>0</surface_radius>
+                            <use_patch_radius>1</use_patch_radius>
+                            <ode>
+                                <slip>0</slip>
+                            </ode>
                         </torsional> -->
                     </friction>
